File: src/5V-Power-Supply/5V-Power-Supply.kicad_sch (KiCad schematic)
At the start: 16 parts, among them U1 LM22672MRE-5.0_NOPB

Commit message: connector
Parts:
- added J?: Conn_01x04_Male, symbol Connector:Conn_01x04_Male
Connections:
- net 5V-BUCK: now also J?.2 (Pin_2)
- net Earth: now also J?.3 (Pin_3)
- net VIN: now also J?.1 (Pin_1), J?.4 (Pin_4)
Changed lines of the file:
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@@
+    (stroke (width 0) (type default) (color 0 0 0 0))
+  )
+  (wire (pts (xy 251.46 58.42) (xy 256.54 58.42))
     (stroke (width 0) (type default) (color 0 0 0 0))
   )
@@
     (stroke (width 0) (type default) (color 0 0 0 0))
   )
+  (wire (pts (xy 251.46 50.8) (xy 256.54 50.8))
+    (stroke (width 0) (type default) (color 0 0 0 0))
+  )
   (wire (pts (xy 153.67 73.66) (xy 163.83 73.66))
     (stroke (width 0) (type default) (color 0 0 0 0))
@@
     (stroke (width 0) (type default) (color 0 0 0 0))
   )
+  (wire (pts (xy 251.46 53.34) (xy 256.54 53.34))
+    (stroke (width 0) (type default) (color 0 0 0 0))
+  )
+  (wire (pts (xy 251.46 55.88) (xy 270.51 55.88))
+    (stroke (width 0) (type default) (color 0 0 0 0))
+  )
   (wire (pts (xy 246.38 110.49) (xy 246.38 115.57))
     (stroke (width 0) (type default) (color 0 0 0 0))
@@
   )
   (wire (pts (xy 231.14 85.09) (xy 231.14 90.17))
+    (stroke (width 0) (type default) (color 0 0 0 0))
+  )
+  (wire (pts (xy 270.51 55.88) (xy 270.51 60.96))
     (stroke (width 0) (type default) (color 0 0 0 0))
   )
@@
     )
   )
+  (global_label "5V-BUCK" (shape input) (at 256.54 53.34 0) (fields_autoplaced)
+    (effects (font (size 1.27 1.27)) (justify left))
+    (property "Intersheet References" "${INTERSHEET_REFS}" (id 0) (at 267.9641 53.2606 0)
+      (effects (font (size 1.27 1.27)) (justify left) hide)
+    )
+  )
   (global_label "V_HEAD" (shape input) (at 68.58 68.58 180) (fields_autoplaced)
     (effects (font (size 1.27 1.27)) (justify right))
@@
     )
   )
+  (global_label "V_HEAD" (shape input) (at 256.54 58.42 0) (fields_autoplaced)
+    (effects (font (size 1.27 1.27)) (justify left))
+    (property "Intersheet References" "${INTERSHEET_REFS}" (id 0) (at 265.8474 58.4994 0)
+      (effects (font (size 1.27 1.27)) (justify left) hide)
+    )
+  )
+  (global_label "VIN" (shape input) (at 256.54 50.8 0) (fields_autoplaced)
+    (effects (font (size 1.27 1.27)) (justify left))
+    (property "Intersheet References" "${INTERSHEET_REFS}" (id 0) (at 261.9769 50.7206 0)
+      (effects (font (size 1.27 1.27)) (justify left) hide)
+    )
+  )
   (global_label "5V-BUCK" (shape input) (at 256.54 85.09 0) (fields_autoplaced)
     (effects (font (size 1.27 1.27)) (justify left))
@@
     (pin "1")
     (pin "2")
+  )
+  (symbol (lib_id "Connector:Conn_01x04_Male") (at 246.38 53.34 0) (unit 1)
+    (in_bom yes) (on_board yes) (fields_autoplaced)
+    (property "Reference" "J?" (id 0) (at 247.015 45.72 0))
+    (property "Value" "Conn_01x04_Male" (id 1) (at 247.015 48.26 0))
+    (property "Footprint" "" (id 2) (at 246.38 53.34 0)
+      (effects (font (size 1.27 1.27)) hide)
+    )
+    (property "Datasheet" "~" (id 3) (at 246.38 53.34 0)
+      (effects (font (size 1.27 1.27)) hide)
+    )
+    (pin "1")
+    (pin "2")
+    (pin "3")
+    (pin "4")
   )
   (symbol (lib_id "5V-Power-Supply1:CAP_0603") (at 231.14 93.98 90) (unit 1)
@@
     (pin "1")
   )
+  (symbol (lib_id "5V-Power-Supply1:Earth") (at 270.51 60.96 0) (unit 1)
+    (in_bom yes) (on_board yes) (fields_autoplaced)
+    (property "Reference" "#PWR?" (id 0) (at 270.51 67.31 0)
+      (effects (font (size 1.27 1.27)) hide)
+    )
+    (property "Value" "Earth" (id 1) (at 270.51 64.77 0)
+      (effects (font (size 1.27 1.27)) hide)
+    )
+    (property "Footprint" "" (id 2) (at 270.51 60.96 0)
+      (effects (font (size 1.27 1.27)) hide)
+    )
+    (property "Datasheet" "" (id 3) (at 270.51 60.96 0)
+      (effects (font (size 1.27 1.27)) hide)
+    )
+    (pin "1")
+  )
   (symbol (lib_id "5V-Power-Supply1:TP") (at 189.23 102.87 0) (unit 1)
     (in_bom yes) (on_board yes) (fields_autoplaced)
@@
       (reference "#PWR06") (unit 1) (value "Earth") (footprint "")
     )
+    (path "/f83d8039-2229-4e70-97d8-88ab97334476"
+      (reference "#PWR?") (unit 1) (value "Earth") (footprint "")
+    )
     (path "/e1e8ab93-53e2-49b4-80f5-4568cb3bae24"
       (reference "C1") (unit 1) (value "68uF") (footprint "")
@@
       (reference "D3") (unit 1) (value "SML-LX1206GC-TR") (footprint "")
     )
+    (path "/0750ed2c-08fe-4122-bdf1-d2051711ce7c"
+      (reference "J?") (unit 1) (value "Conn_01x04_Male") (footprint "")
+    )
     (path "/83df1cb6-463f-4373-8105-981cc8fe8190"

Commit message: initial layout
Parts:
- removed J?: Conn_01x04_Male, symbol Connector:Conn_01x04_Male
- added P1, P2: 0901471110, Connector_PinHeader_1.00mm:PinHeader_1x04_P1.00mm_Horizontal, symbol 5V-Power-Supply1:0901471110
- C1: footprint (none) -> 5V-Power_supply1:EEEFPV680XAP
- C2, C3, C4, C6: footprint (none) -> 5V-Power_supply1:CAP_0603
- C5: footprint (none) -> 5V-Power_supply1:CAP_EEEFP1E151AL
- D1, D3: footprint (none) -> 5V-Power_supply1:SML-LX1206GC-TR
- D2: footprint SOD-123FL_MCC -> 5V-Power_supply1:RB160VAM-60TR
- L1: value CBC3225T220KR -> 33uH; footprint (none) -> 5V-Power_supply1:CBC3225T220KR
- R1, R2: footprint (none) -> 5V-Power_supply1:RES_0603
- TP1, TP2, TP3: footprint (none) -> 5V-Power_supply1:TP
- U1: footprint (none) -> 5V-Power_supply1:LM22672MRE-5.0_NOPB
Connections:
- net 5V-BUCK: now also P2.1
- net Earth: now also P1.2, P1.3, P1.4, P2.2, P2.3, P2.4
- net VIN: now also P1.1
